File: hardware/kicad8.0/IN13-Device.kicad_pcb (KiCad board)
At the start: 2 copper layers, 38.1 x 43.1 mm, 8 parts, among them J1 PINHD_1x3_Female, Q2 MMBTA42, U2 STI3508

Commit message: esp32c6 module
Parts:
- added T1: Transformer_1P_1S, IN13-Device:EE0504S, F.Cu at (83.7, 44.2)
- added U4: ESP32-C6-MINI-1/U, PCM_Espressif:ESP32-C6-MINI-1U, F.Cu at (73.2, 45.3)

Commit message: progress
Parts:
- added C10: 1u, Capacitor_SMD:C_0805_2012Metric, F.Cu at (80.7, 75.5)
- added C11: 1u, Capacitor_SMD:C_0805_2012Metric, F.Cu at (59.1, 74.1)
- added C5: 10u, Capacitor_SMD:C_0805_2012Metric, F.Cu at (79.4, 50.6)
- added C6: 1u, Capacitor_SMD:C_0805_2012Metric, F.Cu at (79.4, 52.6)
- added C7: 1u, Capacitor_SMD:C_0805_2012Metric, F.Cu at (79.4, 41.4)
- added C8: 10u, Capacitor_SMD:C_0805_2012Metric, F.Cu at (79.4, 43.7)
- added C9: 22u, Capacitor_SMD:C_0805_2012Metric, F.Cu at (79.4, 46.0)
- added D2: D_Schottky, Diode_SMD:D_0805_2012Metric, F.Cu at (83.6, 51.7)
- added J2: AudioJack3, Connector_Audio:Jack_3.5mm_CUI_SJ1-3523N_Horizontal, F.Cu at (87.8, 67.8)
- added J3: PINHD_1x4_Male, Connector_PinHeader_2.54mm:PinHeader_1x04_P2.54mm_Vertical, F.Cu at (45.5, 65.5)
- added J4: USB_C_Receptacle_USB2.0_16P, Connector_USB:USB_C_Receptacle_HCTL_HC-TYPE-C-16P-01A, F.Cu at (89.8, 54.3)
- added R1: 1M, Resistor_SMD:R_0805_2012Metric, F.Cu at (62.4, 52.0)
- added R10: 5.1K, Resistor_SMD:R_0603_1608Metric, F.Cu at (90.2, 60.6)
- added R2: 5k, Resistor_SMD:R_0805_2012Metric, F.Cu at (62.3, 49.3)
- added R3: 10k, Resistor_SMD:R_0805_2012Metric, F.Cu at (62.7, 70.9)
- added R4: 330, Resistor_SMD:R_0805_2012Metric, F.Cu at (57.0, 57.3)
- added R5: 220k, Resistor_SMD:R_1206_3216Metric, F.Cu at (62.1, 64.0)
- added R6: 10k, Resistor_SMD:R_0805_2012Metric, F.Cu at (84.4, 75.5)
- added R7: 10k, Resistor_SMD:R_0805_2012Metric, F.Cu at (63.5, 74.1)
- added R8: 10k, Resistor_SMD:R_0805_2012Metric, F.Cu at (61.3, 74.1)
- added R9: 5.1K, Resistor_SMD:R_0603_1608Metric, F.Cu at (86.8, 60.6)
- added RV1: 2k, PCM_Potentiometer_SMD_AKL:Potentiometer_Bourns_TC33X_Vertical, F.Cu at (56.9, 53.0)
- added RV2: 10k, PCM_Potentiometer_SMD_AKL:Potentiometer_Bourns_TC33X_Vertical, F.Cu at (66.4, 43.8)
- added U1: LM358, Package_SO:SOIC-8-1EP_3.9x4.9mm_P1.27mm_EP2.41x3.81mm, F.Cu at (57.5, 65.5)
- added U3: LD1117S33TR_SOT223, Package_TO_SOT_THT:TO-220-3_Horizontal_TabDown, B.Cu at (82.8, 43.5)
- C1, C2, C4: footprint Capacitor_THT:C_Disc_D3.0mm_W2.0mm_P2.50mm -> Capacitor_SMD:C_0805_2012Metric
- C3: footprint Capacitor_THT:C_Disc_D3.0mm_W2.0mm_P2.50mm -> Capacitor_SMD:C_1210_3225Metric
- moved U4 32.6 mm to (71.6, 77.9), turned to 180 degrees
- moved U2 26.8 mm to (73.4, 44.0), turned to 90 degrees
- moved C1 25.0 mm to (79.4, 48.3)
- moved D1 24.6 mm to (67.0, 53.2), turned to 90 degrees
- moved C2 22.2 mm to (79.4, 54.9)
- moved Q2 21.8 mm to (61.2, 59.1), turned to -90 degrees
- moved C3 20.1 mm to (62.1, 55.2)
- moved T1 12.7 mm to (73.1, 51.2), turned to 90 degrees
- moved C4 9.80 mm to (57.0, 59.9), turned to 180 degrees
- moved J1 0.79 mm to (65.5, 59.2)
Connections:
- C1 pad 2: +5V -> +3.3V
- C2 pad 1: +5V -> +3.3V
- T1 pad 4: +5V -> +3.3V
- T1 pad 6: +5V -> +3.3V
- U2 pad 5: +5V -> +3.3V
- U4 pad 17: unconnected-(U4-GPIO12/USB_D--Pad17) -> D-
- U4 pad 18: unconnected-(U4-GPIO13/USB_D+-Pad18) -> D+
- U4 pad 22: HVEN -> Net-(U4-GPIO8)
- U4 pad 23: PWM -> BOOT
- U4 pad 28: unconnected-(U4-GPIO22-Pad28) -> PWM
- U4 pad 29: unconnected-(U4-GPIO23-Pad29) -> HVEN
- U4 pad 30: unconnected-(U4-U0RXD/GPIO17-Pad30) -> RX
- U4 pad 31: unconnected-(U4-U0TXD/GPIO16-Pad31) -> TX
- U4 pad 8: unconnected-(U4-EN/CHIP_PU-Pad8) -> Net-(U4-EN/CHIP_PU)
Other:
- outline, holes or cut-outs redrawn
