File: hardware/kicad8.0/IN13-Device.kicad_sch (KiCad schematic)
At the start: 16 parts, among them J1 PINHD_1x3_Female, Q1 Q_NMOS_DGS, Q2 MMBTA42, T1 Transformer_1P_1S

Commit message: finished basic schematic
Parts:
- removed Q1: Q_NMOS_DGS, symbol Device:Q_NMOS_DGS
- removed R1, R6: 10k, symbol Device:R
- added R3: 10k, symbol Device:R
- added U1: LM358, symbol Amplifier_Operational:LM358
- added U2: STI3508, Package_TO_SOT_SMD:SOT-23-6, symbol IN13-Device:STI3508
- added U3: XIAO-ESP32-C3-DIP, Module:MOUDLE14P-XIAO-DIP-SMD, symbol Xiao:XIAO-ESP32-C3-DIP
- R4: value 10k -> 330
- RV1: value R_Potentiometer -> 2k
- renumbered R2 to R1, R3 to R2
Connections:
- net +5V: now also U1.8 (V+), U2.5 (VIN), U3.14 (VBUS)
- net GND: now also RV1.2, U1.4 (V-), U2.2 (GND), U3.13 (GND); no longer R4.2
- net PWM: now also R3.2, U3.1 (GPIO2/A0/D0)
- net at T1.2 (AB): now also U2.1 (LX)
- net HV: now reaches C3.2, D1.1 (K), J1.1, R1.1
- net at RV1.1: now also R4.2
- net HVMON: no longer names the net of R1.2, R2.1
- net HVMON: now also U2.3 (FB)
- net OPIN+: no longer names the net of C4.1
- net OPIN+: now also R3.1, U1.3 (+)
- net OPIN-: no longer names the net of Q2.2 (E), R4.1
- net OPIN-: now also U1.2 (-)
- net OPOUT: no longer names the net of Q2.1 (B)
- net OPOUT: now also U1.1
- new net HVEN: U2.4 (EN), U3.5 (GPIO6/D4/SDA)
- no-connect marks 0 -> 14
Other:
- title: (none) -> IN-13 Device
- moved on the sheet: C1, C2, C4, D1, J1, Q2, R1, R2, R4, R5, RV1, T1

Commit message: esp32c6 module
Parts:
- removed U3: XIAO-ESP32-C3-DIP, Module:MOUDLE14P-XIAO-DIP-SMD, symbol Xiao:XIAO-ESP32-C3-DIP
- added U4: ESP32-C6-MINI-1/U, PCM_Espressif:ESP32-C6-MINI-1U, symbol PCM_Espressif:ESP32-C6-MINI-1/U
- T1: footprint (none) -> IN13-Device:EE0504S; symbol Device:Transformer_1P_1S -> IN13-Device:EE0504S_Transformer
Connections:
- net +5V: now also T1.6 (SB); no longer T1.1 (AA)
- net GND: now also U4.1 (GND), U4.11 (GND), U4.14 (GND), U4.2 (GND), U4.36 (GND), U4.37 (GND), U4.38 (GND), U4.39 (GND), U4.40 (GND), U4.41 (GND), U4.42 (GND), U4.43 (GND), U4.44 (GND), U4.45 (GND), U4.46 (GND), U4.47 (GND), U4.48 (GND), U4.49 (GND), U4.50 (GND), U4.51 (GND), U4.52 (GND), U4.53 (GND)
- net HVEN: now also U4.22 (GPIO8)
- net PWM: now also U4.23 (GPIO9)
- net at U2.1 (LX): now also T1.1 (AB); no longer T1.2 (AB)
- net at D1.2 (A): now also T1.5 (SA); no longer T1.3 (SA)
- new net +3.3V: U4.3 (3V3)
- new net SIGNAL: U4.12 (GPIO0/ADC1_CH0/XTAL_32K_P)
- no-connect marks 14 -> 23
Other:
- moved on the sheet: C1, C2, C3, C4, D1, J1, Q2, R1, R2, R3, R4, R5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

Commit message: progress
Parts:
- added C10, C11, C6, C7: 1u, Capacitor_SMD:C_0805_2012Metric, symbol Device:C
- added C5, C8: 10u, Capacitor_SMD:C_0805_2012Metric, symbol Device:C
- added C9: 22u, Capacitor_SMD:C_0805_2012Metric, symbol Device:C
- added D2: D_Schottky, Diode_SMD:D_0805_2012Metric, symbol Device:D_Schottky
- added J2: AudioJack3, Connector_Audio:Jack_3.5mm_CUI_SJ1-3523N_Horizontal, symbol Connector_Audio:AudioJack3
- added J3: PINHD_1x4_Male, Connector_PinHeader_2.54mm:PinHeader_1x04_P2.54mm_Vertical, symbol PCM_SL_Pin_Headers:PINHD_1x4_Male
- added J4: USB_C_Receptacle_USB2.0_16P, Connector_USB:USB_C_Receptacle_HCTL_HC-TYPE-C-16P-01A, symbol Connector:USB_C_Receptacle_USB2.0_16P
- added R10, R9: 5.1K, Resistor_SMD:R_0603_1608Metric, symbol Device:R
- added R6, R7, R8: 10k, Resistor_SMD:R_0805_2012Metric, symbol Device:R
- added RV2: 10k, PCM_Potentiometer_SMD_AKL:Potentiometer_Bourns_TC33X_Vertical, symbol Device:R_Potentiometer
- added U3: LD1117S33TR_SOT223, Package_TO_SOT_THT:TO-220-3_Horizontal_TabDown, symbol Regulator_Linear:LD1117S33TR_SOT223
- C1, C2, C4: footprint Capacitor_THT:C_Disc_D3.0mm_W2.0mm_P2.50mm -> Capacitor_SMD:C_0805_2012Metric
- C3: footprint Capacitor_THT:C_Disc_D3.0mm_W2.0mm_P2.50mm -> Capacitor_SMD:C_1210_3225Metric
- R1, R3, R4: footprint (none) -> Resistor_SMD:R_0805_2012Metric
- R2: value 10k -> 5k; footprint (none) -> Resistor_SMD:R_0805_2012Metric
- R5: footprint (none) -> Resistor_SMD:R_1206_3216Metric
- RV1: footprint (none) -> PCM_Potentiometer_SMD_AKL:Potentiometer_Bourns_TC33X_Vertical
- U1: footprint (none) -> Package_SO:SOIC-8-1EP_3.9x4.9mm_P1.27mm_EP2.41x3.81mm
Connections:
- net +5V is gone; now on net +3.3V: C1.2, C2.1, T1.4 (AA), T1.6 (SB), U1.8 (V+), U2.5 (VIN)
- net +3.3V: now also J2.T, J3.1, R6.1, R7.2, R8.2
- net GND: now also RV1.3, C10.2, C11.2, C5.2, C6.2, C7.2, C8.2, C9.2, J2.S, J3.4, J4.A1 (GND), J4.A12 (GND), J4.B1 (GND), J4.B12 (GND), J4.S1 (SHIELD), R10.2, R9.2, U3.1 (GND)
- net HV: now also R1.2; no longer R1.1
- net HVEN: now also U4.29 (GPIO23); no longer U4.22 (GPIO8)
- net PWM: now also U4.28 (GPIO22); no longer U4.23 (GPIO9)
- net SIGNAL: now also J2.R
- net D-: now reaches U4.17 (GPIO12/USB_D-)
- net D-: now also J4.A7 (D-), J4.B7 (D-)
- net D+: now reaches U4.18 (GPIO13/USB_D+)
- net D+: now also J4.A6 (D+), J4.B6 (D+)
- net RX: now reaches U4.30 (U0RXD/GPIO17)
- net RX: now also J3.3
- net TX: now reaches U4.31 (U0TXD/GPIO16)
- net TX: now also J3.2
- net at U4.8 (EN/CHIP_PU): now also C10.1, R6.2
- new net: R1.1, RV2.1, U2.3 (FB)
- new net: R2.1, RV2.2, RV2.3
- new net: R7.1, U4.22 (GPIO8)
- new net: J4.A5 (CC1), R10.1
- new net: J4.B5 (CC2), R9.1
- new net +3V3: C7.1, C8.1, C9.1, U3.2 (VO)
- new net BOOT: C11.1, R8.1, U4.23 (GPIO9)
- new net VBUS: D2.2 (A), J4.A4 (VBUS), J4.A9 (VBUS), J4.B4 (VBUS), J4.B9 (VBUS)
- new net VIN: C5.1, C6.1, D2.1 (K), U3.3 (VI)
- no-connect marks 23 -> 18
Other:
- note added: "Cathode Control"
- note added: "MCU"
- note added: "Power"
- moved on the sheet: C1, C2, C3, C4, J1, Q2, R1, R3, R4, R5, RV1, T1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
