File: hardware/kicad8.0/IN13-Nixie-Device.kicad_pcb (KiCad board)
At the start: 2 copper layers, 38.1 x 43.1 mm, 40 parts, among them J1 PINHD_1x3_Female, J2 AudioJack3, J3 PINHD_1x4_Male, J4 USB_C_Receptacle_USB2.0_16P, J5 PINHD_1x4_Male, Q2 MMBTA42, SW1 SW_Push, SW3 SW_Push, T1 Transformer_1P_1S, U1 LM358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

Commit message: pcb revision
Parts:
- added D3: LED, LED_SMD:LED_0603_1608Metric, F.Cu at (63.2, 69.3)
- added R12: 220, Resistor_SMD:R_0603_1608Metric, F.Cu at (66.3, 68.5)
- moved TP2 26.0 mm to (70.5, 41.5)
- moved C11 4.33 mm to (62.3, 76.3), turned to 180 degrees
- moved R3 3.54 mm to (61.2, 67.5)
- moved R8 2.73 mm to (62.3, 74.7), turned to 180 degrees
- moved R7 1.17 mm to (62.3, 73.0), turned to 180 degrees
- moved R5 0.45 mm to (61.8, 61.8)
- moved TP1 0.37 mm to (61.2, 70.9)
- moved R6 0.10 mm to (78.8, 75.0)
- turned T1 to 0 degrees
Connections:
- T1 pad 5: Net-(D1-A) -> GND
- T1 pad 6: +3.3V -> Net-(D1-A)
- TP2 pad 1: HVEN -> Net-(U2-FB)
Routing:
- net BOOT: track 21.6 -> 13.7 mm
- net Net-(T1-AB): track 8.35 -> 3.53 mm
- net Net-(U1A-+): track 16.3 -> 12.6 mm
- net GND: track 126.7 -> 123.3 mm
- net PWM: track 3.92 -> 6.38 mm
- net Net-(D3-A): track 0.00 -> 2.28 mm
- net Net-(U2-FB): track 14.2 -> 16.4 mm
- net Net-(D1-A): track 4.16 -> 6.03 mm
- net +3.3V: track 139.7 -> 138.2 mm
- net HVEN: track 41.4 -> 40.6 mm, vias 0 -> 2
- net VBUS: track 13.3 -> 12.6 mm
- net TX: track 11.6 -> 10.9 mm
