File: hardware/kicad10.0/IN13-Nixie-Device.kicad_pcb (KiCad board)
At the start: 2 copper layers, 38.1 x 43.1 mm, 44 parts, among them J1 PINHD_1x3_Female, J2 AudioJack3, J3 USB_C_Receptacle_USB2.0_16P, J4 PINHD_1x4_Male, J5 PINHD_1x4_Male, Q1 MMBTA42, SW1 SW_Push, SW2 SW_Push, T1 EE0504S 1:10, U1 LM358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

Commit message: schematic and layour rework start
Parts:
- removed C1: 1u, Capacitor_SMD:C_0603_1608Metric
- removed C10, C7: 1u, Capacitor_SMD:C_0805_2012Metric
- removed C11, C8: 10u, Capacitor_SMD:C_0805_2012Metric
- removed C5: 1u 200V, Capacitor_SMD:C_1210_3225Metric
- removed C6: 0.22u 200V, Capacitor_SMD:C_1210_3225Metric
- removed D1: US1G, Diode_SMD:D_SMA
- removed R10: 4.3k, Resistor_SMD:R_0805_2012Metric
- removed R8: 48K, Resistor_SMD:R_0805_2012Metric
- removed R9: 1M, Resistor_SMD:R_0805_2012Metric
- removed T1: EE0504S 1:10, IN13-Nixie-Device:EE0504S_Wide
- removed TP3: TestPoint, TestPoint:TestPoint_Pad_1.0x1.0mm
- removed U3: FP6291, Package_TO_SOT_SMD:SOT-23-6
- added U11: HV Module, IN13-Nixie-Device:AliExpress_HV_Module, F.Cu at (71.6, 47.6)
- J2, J3: moved to B.Cu
- U4: value AMS1117-3.3 -> AP2112K-3.3; footprint Package_TO_SOT_SMD:SOT-223-3_TabPin2 -> Package_TO_SOT_SMD:SOT-23-5
- moved C12 32.0 mm to (82.0, 74.4), turned to 0 degrees
- moved U4 22.7 mm to (82.1, 71.3), turned to 180 degrees
- moved D2 20.9 mm to (83.6, 64.6)
- moved R11 19.7 mm to (84.5, 55.3), turned to 90 degrees
- moved J3 16.0 mm to (89.8, 69.2), turned to -90 degrees
- moved R7 15.0 mm to (81.0, 65.2)
- moved R13 14.0 mm to (88.9, 70.9), turned to 0 degrees
- moved C9 12.9 mm to (82.0, 68.1), turned to 180 degrees
- moved J2 12.5 mm to (87.8, 55.3), turned to -90 degrees
- moved TP2 10.9 mm to (65.6, 67.2)
- moved R12 10.5 mm to (88.9, 67.9), turned to 0 degrees
- moved R1 7.53 mm to (66.3, 55.7), turned to 180 degrees
- moved C2 1.60 mm to (57.2, 58.7)
- moved R4 1.37 mm to (57.0, 56.0)
- moved RV1 1.29 mm to (58.4, 51.3)
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Connections:
- J1 pad 1: HV -> Net-(J1-Pad1)
- J1 pad 3: Net-(J1-Pad3) -> HV
- J3 pad S1: GND -> (no net)
- R1 pad 1: Net-(J1-Pad3) -> GND
- R1 pad 2: GND -> Net-(J1-Pad1)
- U4 pad 1: GND -> VBUS
- U4 pad 2: +3.3V -> GND
Routing:
- net +3.3V: track 112.8 -> 47.4 mm, vias 3 -> 2
- net GND: track 124.3 -> 77.1 mm, vias 20 -> 7
- net HVEN: track 40.9 -> 0.00 mm, vias 2 -> 0
- net D+: track 32.3 -> 0.00 mm, vias 2 -> 0
- net D-: track 31.2 -> 0.04 mm, vias 2 -> 0
- net HV: track 20.2 -> 0.00 mm
- net VBUS: track 34.5 -> 17.1 mm, vias 0 -> 3
- net Net-(U3-FB): track 10.8 -> 0.00 mm
- net Net-(U3-OC): track 9.35 -> 0.00 mm
- net SIGNAL: track 8.87 -> 0.00 mm
- net Net-(J3-CC2): track 10.8 -> 2.03 mm, vias 2 -> 1
- net EN: track 27.3 -> 18.8 mm, vias 2 -> 0
- net Net-(D1-A): track 5.71 -> 0.00 mm
- net Net-(Q1-E): track 8.13 -> 12.7 mm
- net Net-(Q1-B): track 5.16 -> 9.71 mm
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Other:
- outline, holes or cut-outs redrawn

Commit message: revision passing DRC
Parts:
- removed D2: LED, LED_SMD:LED_0603_1608Metric
- removed R7: 220, Resistor_SMD:R_0603_1608Metric
- added D3: LED, LED_SMD:LED_0603_1608Metric, F.Cu at (82.3, 42.8)
- added R14: 220, Resistor_SMD:R_0603_1608Metric, F.Cu at (82.3, 46.3)
- added TP4: TestPoint, TestPoint:TestPoint_Pad_1.0x1.0mm, F.Cu at (82.8, 53.0)
- J4, J5: footprint SharedCustom:Pads_1x4_2.54mm -> IN13-Nixie-Device:Pads_1x4_2.54mm
- moved TP2 6.27 mm to (62.1, 62.0)
- moved R11 3.68 mm to (82.2, 58.2), turned to 180 degrees
- moved C2 2.22 mm to (57.5, 56.5)
- moved R4 2.16 mm to (57.5, 53.9)
- moved TP1 1.25 mm to (62.3, 70.2)
- moved U1 0.95 mm to (57.8, 62.4), turned to -90 degrees
- moved RV1 0.91 mm to (58.3, 50.4), turned to 180 degrees
- moved Q1 0.68 mm to (62.0, 57.4), turned to -90 degrees
- moved C9 0.57 mm to (82.6, 68.1)
- moved U4 0.57 mm to (82.7, 71.3)
- moved C12 0.57 mm to (82.6, 74.4)
- moved R1 0.49 mm to (66.7, 55.4)
Connections:
- U2 pad 12: unconnected-(U2-GPIO0/ADC1_CH0/XTAL_32K_P-Pad12) -> HVEN
- U2 pad 20: HVEN -> unconnected-(U2-GPIO15-Pad20)
Routing:
- net HVEN: track 0.00 -> 34.0 mm
- net SIGNAL: track 0.00 -> 31.4 mm
- net GND: track 77.1 -> 104.5 mm, vias 7 -> 17
- net +3.3V: track 47.4 -> 71.8 mm, vias 2 -> 3
- net D+: track 0.00 -> 19.9 mm, vias 0 -> 1
- net HV: track 0.00 -> 19.4 mm, vias 0 -> 1
- net D-: track 0.04 -> 19.2 mm, vias 0 -> 1
- net VBUS: track 17.1 -> 32.8 mm
- net EN: track 18.8 -> 27.3 mm, vias 0 -> 2
- net Net-(R4-Pad2): track 0.00 -> 4.75 mm
- net Net-(Q1-B): track 9.71 -> 5.07 mm
- net Net-(Q1-E): track 12.7 -> 8.29 mm
- net TCK: track 9.75 -> 14.1 mm
- net Net-(J1-Pad1): track 0.00 -> 3.91 mm
- net TDO: track 10.5 -> 13.2 mm
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
Commit message: final rev 0.4
Parts:
- added TP5: TestPoint, TestPoint:TestPoint_Pad_1.0x1.0mm, F.Cu at (66.6, 68.1)
- moved R1 0.98 mm to (67.7, 55.6), turned to -160 degrees
- moved R3 0.96 mm to (62.0, 67.0)
- moved D3 0.39 mm to (82.6, 42.8)
- moved R14 0.39 mm to (82.6, 46.3)
- moved C12 0.29 mm to (82.6, 74.1)
- moved C9 0.29 mm to (82.6, 67.8)
- moved U4 0.29 mm to (82.7, 71.0)
- moved TP1 0.22 mm to (62.0, 70.2), turned to 90 degrees
- moved C3 0.18 mm to (78.8, 71.8)
- turned U11 to 0 degrees
Connections:
- J3 pad SH: (no net) -> GND
- U2 pad 20: unconnected-(U2-GPIO15-Pad20) -> Net-(U2-GPIO15)
Routing:
- net GND: track 104.5 -> 114.7 mm, vias 17 -> 14
- net VBUS: track 32.8 -> 27.7 mm
- net Net-(U2-GPIO15): track 0.00 -> 3.86 mm
- net HV: track 19.4 -> 16.4 mm
- net HVEN: track 34.0 -> 33.3 mm
- net Net-(Q1-B): track 5.07 -> 4.50 mm
- net +3.3V: track 71.8 -> 71.2 mm
- net Net-(U1A-+): track 12.5 -> 11.9 mm
Other:
- board text added: "IN-13 Nixie Device"
- board text added: "rev 0.4"
