File: hardware/kicad10.0/IN13-Nixie-Device.kicad_sch (KiCad schematic)
At the start: 44 parts, among them J1 PINHD_1x3_Female, J2 AudioJack3, J3 USB_C_Receptacle_USB2.0_16P, J4 PINHD_1x4_Male, J5 PINHD_1x4_Male, Q1 MMBTA42, SW1 SW_Push, SW2 SW_Push, T1 EE0504S 1:10, U1 LM358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

Commit message: pivot to hv module, kicad 10.0
Parts:
- added U11: HV Module, Nixie:AliExpress_HV_Module, symbol IN13-Nixie-Device:AliExpress_HV_Module
Connections:
- net GND: now also U11.3 (Gnd)
- net HV: now also U11.4 (Vout)
- net HVEN: now also U11.2 (EN)
- net VBUS: now also U11.1 (Vin)
Other:
- note added: "TODO: Design boost circuit external, using module for now"
- moved on the sheet: C5, C6, D1, D2, R10, R7, R8, R9, T1, TP2, TP3, U3

Commit message: schematic fixes
Parts:
- U11: footprint Nixie:AliExpress_HV_Module -> IN13-Nixie-Device:AliExpress_HV_Module
Connections:
- net GND: now also J3.SH (SHIELD), R1.1; no longer J3.S1 (SHIELD), R1.2
- net HV: now also J1.3; no longer J1.1
- new net: J1.1, R1.2
Changed lines of the file:
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@@
 	(wire
 		(pts
-			(xy 173.99 34.29) (xy 176.53 34.29)
+			(xy 173.99 34.29) (xy 175.26 34.29)
 		)
 		(stroke
@@
 	(wire
 		(pts
+			(xy 161.29 34.29) (xy 160.02 34.29)
+		)
+		(stroke
+			(width 0)
+			(type default)
+		)
+	)
+	(wire
+		(pts
 			(xy 106.68 69.85) (xy 105.41 69.85)
 		)
@@
 	(wire
 		(pts
-			(xy 177.8 163.83) (xy 177.8 166.37)
+			(xy 160.02 34.29) (xy 160.02 35.56)
 		)
 		(stroke
@@
 	(wire
 		(pts
-			(xy 92.71 49.53) (xy 91.44 49.53)
+			(xy 177.8 163.83) (xy 177.8 166.37)
 		)
 		(stroke
@@
 	(wire
 		(pts
-			(xy 101.6 30.48) (xy 102.87 30.48)
+			(xy 92.71 49.53) (xy 91.44 49.53)
 		)
 		(stroke
@@
 	(wire
 		(pts
-			(xy 138.43 163.83) (xy 138.43 166.37)
+			(xy 101.6 30.48) (xy 102.87 30.48)
 		)
 		(stroke
@@
 	(wire
 		(pts
-			(xy 186.69 34.29) (xy 186.69 36.83)
+			(xy 138.43 163.83) (xy 138.43 166.37)
 		)
 		(stroke
@@
 	(wire
 		(pts
-			(xy 184.15 34.29) (xy 186.69 34.29)
-		)
-		(stroke
-			(width 0)
-			(type default)
-		)
-	)
-	(wire
-		(pts
 			(xy 21.59 45.72) (xy 21.59 46.99)
 		)
@@
 	(wire
 		(pts
-			(xy 167.64 34.29) (xy 168.91 34.29)
-		)
-		(stroke
-			(width 0)
-			(type default)
-		)
-	)
-	(wire
-		(pts
 			(xy 280.67 181.61) (xy 280.67 182.88)
 		)
@@
 		)
 	)
-	(global_label "D+"
+	(global_label "HV"
 		(shape input)
-		(at 95.25 154.94 0)
+		(at 175.26 34.29 0)
 		(fields_autoplaced yes)
 		(effects
@@
 		)
 		(property "Intersheetrefs" "${INTERSHEET_REFS}"
-			(at 101.0776 154.94 0)
+			(at 180.6643 34.29 0)
 			(hide yes)
 			(show_name no)
@@
 		)
 	)
-	(global_label "HV"
+	(global_label "D+"
 		(shape input)
-		(at 167.64 34.29 180)
+		(at 95.25 154.94 0)
 		(fields_autoplaced yes)
 		(effects
@@
 				(size 1.27 1.27)
 			)
-			(justify right)
+			(justify left)
 		)
 		(property "Intersheetrefs" "${INTERSHEET_REFS}"
-			(at 162.2357 34.29 0)
+			(at 101.0776 154.94 0)
 			(hide yes)
 			(show_name no)
@@
 					(size 1.27 1.27)
 				)
-				(justify right)
+				(justify left)
 			)
 		)
@@
 	)
 	(symbol
+		(lib_id "power:GND")
+		(at 160.02 35.56 0)
+		(unit 1)
+		(body_style 1)
+		(exclude_from_sim no)
+		(in_bom yes)
+		(on_board yes)
+		(in_pos_files yes)
+		(dnp no)
+		(property "Reference" "#PWR05"
+			(at 160.02 41.91 0)
+			(hide yes)
+			(show_name no)
+			(do_not_autoplace no)
+			(effects
+				(font
+					(size 1.27 1.27)
+				)
+			)
+		)
+		(property "Value" "GND"
+			(at 160.02 39.37 0)
+			(show_name no)
+			(do_not_autoplace no)
+			(effects
+				(font
+					(size 1.27 1.27)
+				)
+			)
+		)
+		(property "Footprint" ""
+			(at 160.02 35.56 0)
+			(hide yes)
+			(show_name no)
+			(do_not_autoplace no)
+			(effects
+				(font
+					(size 1.27 1.27)
+				)
+			)
+		)
+		(property "Datasheet" ""
+			(at 160.02 35.56 0)
+			(hide yes)
+			(show_name no)
+			(do_not_autoplace no)
+			(effects
+				(font
+					(size 1.27 1.27)
+				)
+			)
+		)
+		(property "Description" "Power symbol creates a global label with name \"GND\" , ground"
+			(at 160.02 35.56 0)
+			(hide yes)
+			(show_name no)
+			(do_not_autoplace no)
+			(effects
+				(font
+					(size 1.27 1.27)
+				)
+			)
+		)
+		(pin "1"
+		)
+		(instances
+			(project "IN13-Nixie-Device"
+				(path "/36cde5b7-6663-4cfe-a0a3-3f17918aab11"
+					(reference "#PWR05")
+					(unit 1)
+				)
+			)
+		)
+	)
+	(symbol
 		(lib_id "Device:R")
 		(at 48.26 140.97 0)
@@
 		(pin "B9"
 		)
-		(pin "S1"
+		(pin "SH"
 		)
 		(instances
@@
 	(symbol
 		(lib_id "power:GND")
-		(at 186.69 36.83 0)
-		(unit 1)
-		(body_style 1)
-		(exclude_from_sim no)
-		(in_bom yes)
-		(on_board yes)
-		(in_pos_files yes)
-		(dnp no)
-		(property "Reference" "#PWR05"
-			(at 186.69 43.18 0)
-			(hide yes)
-			(show_name no)
-			(do_not_autoplace no)
-			(effects
-				(font
-					(size 1.27 1.27)
-				)
-			)
-		)
-		(property "Value" "GND"
-			(at 186.69 40.64 0)
-			(show_name no)
-			(do_not_autoplace no)
-			(effects
-				(font
-					(size 1.27 1.27)
-				)
-			)
-		)
-		(property "Footprint" ""
-			(at 186.69 36.83 0)
-			(hide yes)
-			(show_name no)
-			(do_not_autoplace no)
-			(effects
-				(font
-					(size 1.27 1.27)
-				)
-			)
-		)
-		(property "Datasheet" ""
-			(at 186.69 36.83 0)
-			(hide yes)
-			(show_name no)
-			(do_not_autoplace no)
-			(effects
-				(font
-					(size 1.27 1.27)
-				)
-			)
-		)
-		(property "Description" "Power symbol creates a global label with name \"GND\" , ground"
-			(at 186.69 36.83 0)
-			(hide yes)
-			(show_name no)
-			(do_not_autoplace no)
-			(effects
-				(font
-					(size 1.27 1.27)
-				)
-			)
-		)
-		(pin "1"
-		)
-		(instances
-			(project "IN13-Nixie-Device"
-				(path "/36cde5b7-6663-4cfe-a0a3-3f17918aab11"
-					(reference "#PWR05")
-					(unit 1)
-				)
-			)
-		)
-	)
-	(symbol
-		(lib_id "power:GND")
 		(at 110.49 147.32 0)
 		(unit 1)
@@
 			)
 		)
-		(property "Footprint" "Nixie:AliExpress_HV_Module"
+		(property "Footprint" "IN13-Nixie-Device:AliExpress_HV_Module"
 			(at 156.464 119.634 0)
 			(hide yes)
@@
 	)
 	(symbol
-		(lib_id "Device:R")
-		(at 180.34 34.29 90)
-		(unit 1)
-		(body_style 1)
-		(exclude_from_sim no)
-		(in_bom yes)
-		(on_board yes)
-		(in_pos_files yes)
-		(dnp no)
-		(property "Reference" "R1"
-			(at 181.61 32.004 90)
-			(show_name no)
-			(do_not_autoplace no)
-			(effects
-				(font
-					(size 1.27 1.27)
-				)
-				(justify left)
-			)
-		)
-		(property "Value" "220k"
-			(at 182.626 34.29 90)
-			(show_name no)
-			(do_not_autoplace no)
-			(effects
-				(font
-					(size 1.27 1.27)
-				)
-				(justify left)
-			)
-		)
-		(property "Footprint" "Resistor_SMD:R_1206_3216Metric"
-			(at 180.34 36.068 90)
-			(hide yes)
-			(show_name no)
-			(do_not_autoplace no)
-			(effects
-				(font
-					(size 1.27 1.27)
-				)
-			)
-		)
-		(property "Datasheet" ""
-			(at 180.34 34.29 0)
-			(hide yes)
-			(show_name no)
-			(do_not_autoplace no)
-			(effects
-				(font
-					(size 1.27 1.27)
-				)
-			)
-		)
-		(property "Description" "Resistor"
-			(at 180.34 34.29 0)
-			(hide yes)
-			(show_name no)
-			(do_not_autoplace no)
-			(effects
-				(font
-					(size 1.27 1.27)
-				)
-			)
-		)
-		(pin "2"
-		)
-		(pin "1"
-		)
-		(instances
-			(project "IN13-Nixie-Device"
-				(path "/36cde5b7-6663-4cfe-a0a3-3f17918aab11"
-					(reference "R1")
-					(unit 1)
-				)
-			)
-		)
-	)
-	(symbol
 		(lib_id "power:GND")
 		(at 280.67 182.88 0)
@@
 					(unit 1)
 				)
+			)
+		)
+	)
+	(symbol
+		(lib_id "Device:R")
+		(at 165.1 34.29 90)
+		(unit 1)
+		(body_style 1)
+		(exclude_from_sim no)
+		(in_bom yes)
+		(on_board yes)
+		(in_pos_files yes)
+		(dnp no)
+		(property "Reference" "R1"
+			(at 166.37 32.004 90)
+			(show_name no)
+			(do_not_autoplace no)
+			(effects
+				(font
+					(size 1.27 1.27)
+				)
+				(justify left)
+			)
+		)
+		(property "Value" "220k"
+			(at 167.386 34.29 90)
+			(show_name no)
+			(do_not_autoplace no)
+			(effects
+				(font
+					(size 1.27 1.27)
+				)
+				(justify left)
+			)
+		)
+		(property "Footprint" "Resistor_SMD:R_1206_3216Metric"
+			(at 165.1 36.068 90)
+			(hide yes)
+			(show_name no)
+			(do_not_autoplace no)
+			(effects
+				(font
+					(size 1.27 1.27)
+				)
+			)
+		)
+		(property "Datasheet" ""
+			(at 165.1 34.29 0)
+			(hide yes)
+			(show_name no)
+			(do_not_autoplace no)
+			(effects
+				(font
+					(size 1.27 1.27)
+				)
+			)
+		)
+		(property "Description" "Resistor"
+			(at 165.1 34.29 0)
+			(hide yes)
+			(show_name no)
+			(do_not_autoplace no)
+			(effects
+				(font
+					(size 1.27 1.27)
+				)
+			)
+		)
+		(pin "2"
+		)
+		(pin "1"
+		)
+		(instances
+			(project "IN13-Nixie-Device"
+				(path "/36cde5b7-6663-4cfe-a0a3-3f17918aab11"
+					(reference "R1")
+					(unit 1)
+				)

Commit message: schematic and layour rework start
Parts:
- removed C1: 1u, Capacitor_SMD:C_0603_1608Metric, symbol Device:C
- removed C10, C7: 1u, Capacitor_SMD:C_0805_2012Metric, symbol Device:C
- removed C11, C8: 10u, Capacitor_SMD:C_0805_2012Metric, symbol Device:C
- U4: value AMS1117-3.3 -> AP2112K-3.3; footprint Package_TO_SOT_SMD:SOT-223-3_TabPin2 -> Package_TO_SOT_SMD:SOT-23-5; symbol Regulator_Linear:AMS1117-3.3 -> Regulator_Linear:AP2112K-3.3
Connections:
- net +3.3V: now also U4.5 (VOUT); no longer U4.2 (VO)
- net GND: now also U4.2 (GND); no longer U4.1 (GND)
- net VBUS: now also U4.1 (VIN)
Other:
- moved on the sheet: C12, C9

Commit message: revision passing DRC
Parts:
- added D3: LED, LED_SMD:LED_0603_1608Metric, symbol Device:LED
- added R14: 220, Resistor_SMD:R_0603_1608Metric, symbol Device:R
- added TP4: TestPoint, TestPoint:TestPoint_Pad_1.0x1.0mm, symbol Connector:TestPoint
- C2, C5, C6: symbol PCM_SL_Devices:Capacitor_NP -> Device:C
- J1: symbol PCM_SL_Pin_Headers:PINHD_1x3_Female -> IN13-Nixie-Device:PINHD_1x3_Female
- J4, J5: footprint SharedCustom:Pads_1x4_2.54mm -> IN13-Nixie-Device:Pads_1x4_2.54mm; symbol PCM_SL_Pin_Headers:PINHD_1x4_Male -> IN13-Nixie-Device:PINHD_1x4_Male
- U2: footprint PCM_Espressif:ESP32-C6-MINI-1U -> PCM_Espressif:ESP32-C6-MINI-1
Connections:
- net GND: now also R7.1, R14.1; no longer D2.1 (K)
- net HVEN: now also D2.2 (A), U2.12 (GPIO0/ADC1_CH0/XTAL_32K_P), D3.2 (A); no longer R7.2, U2.20 (GPIO15)
- net SIGNAL: now also TP4.1
- new net: D2.1 (K), R7.2
- new net: D3.1 (K), R14.2
- no-connect marks 14 -> 15
Other:
- note added: "HV Boost Module"
- note added: "TODO: Design/finalize custom boost circuit later, using module for now"
- note removed: "TODO: Design boost circuit external, using module for now"
- moved on the sheet: D1, R10, R8, R9, T1, TP2, TP3, U3

Commit message: final rev 0.4
Parts:
- added TP5: TestPoint, TestPoint:TestPoint_Pad_1.0x1.0mm, symbol Connector:TestPoint
- U2: footprint PCM_Espressif:ESP32-C6-MINI-1 -> PCM_Espressif:ESP32-C6-MINI-1U
Connections:
- net at U2.20 (GPIO15): now also TP5.1
- no-connect marks 15 -> 14
Changed lines of the file:
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@@
 	)
 	(no_connect
-		(at 100.33 87.63)
-	)
-	(no_connect
 		(at 91.44 90.17)
 	)
@@
 			)
 		)
-		(property "Footprint" "PCM_Espressif:ESP32-C6-MINI-1"
+		(property "Footprint" "PCM_Espressif:ESP32-C6-MINI-1U"
 			(at 63.5 120.015 0)
 			(hide yes)
@@
 	)
 	(symbol
+		(lib_id "Connector:TestPoint")
+		(at 100.33 87.63 270)
+		(unit 1)
+		(body_style 1)
+		(exclude_from_sim no)
+		(in_bom yes)
+		(on_board yes)
+		(in_pos_files yes)
+		(dnp no)
+		(property "Reference" "TP5"
+			(at 105.156 87.63 90)
+			(show_name no)
+			(do_not_autoplace no)
+			(effects
+				(font
+					(size 1.27 1.27)
+				)
+				(justify left)
+			)
+		)
+		(property "Value" "TestPoint"
+			(at 109.982 86.868 0)
+			(hide yes)
+			(show_name no)
+			(do_not_autoplace no)
+			(effects
+				(font
+					(size 1.27 1.27)
+				)
+				(justify left)
+			)
+		)
+		(property "Footprint" "TestPoint:TestPoint_Pad_1.0x1.0mm"
+			(at 100.33 92.71 0)
+			(hide yes)
+			(show_name no)
+			(do_not_autoplace no)
+			(effects
+				(font
+					(size 1.27 1.27)
+				)
+			)
+		)
+		(property "Datasheet" ""
+			(at 100.33 92.71 0)
+			(hide yes)
+			(show_name no)
+			(do_not_autoplace no)
+			(effects
+				(font
+					(size 1.27 1.27)
+				)
+			)
+		)
+		(property "Description" "test point"
+			(at 100.33 87.63 0)
+			(hide yes)
+			(show_name no)
+			(do_not_autoplace no)
+			(effects
+				(font
+					(size 1.27 1.27)
+				)
+			)
+		)
+		(pin "1"
+		)
+		(instances
+			(project "IN13-Nixie-Device"
+				(path "/36cde5b7-6663-4cfe-a0a3-3f17918aab11"
+					(reference "TP5")
+					(unit 1)
+				)
+			)
+		)
+	)
+	(symbol
 		(lib_id "power:GND")
 		(at 76.2 30.48 0)
@@
 		(exclude_from_sim no)
 		(in_bom yes)
-		(on_board yes)
+		(on_board no)
 		(in_pos_files yes)
 		(dnp no)
@@
 		(exclude_from_sim no)
 		(in_bom yes)
-		(on_board yes)
+		(on_board no)
 		(in_pos_files yes)
 		(dnp no)
